Commit message: modified:   ros2_ws/log/latest_build 	modified:   ros2_ws/src/my_package/urdf/vehicle.urdf 	modified:   ros2_ws/src/robot_state_publisher/robot_state_publisher/robot_state_publisher_node.py

File: ros2_ws/src/my_package/urdf/vehicle.urdf (robot description, URDF)
Before this commit: robot tiguan, 32 links, 31 joints
Links:
- added link camera_front_wide
Joints:
- added joint base_link_to_camera_front_wide_joint: type fixed, parent base_link, child camera_front_wide, origin xyz=-0.424 0.003 -0.006 rpy=0.245 -1.519 -0.295
